File: 24S_Counter.kicad_pcb (KiCad board)
At the start: 2 copper layers, 0 parts

Commit message: op
Parts:
- added G***: LOGO, LOGO, F.Cu at (113.0, 118.0)
- added H1: MountingHole, MountingHole:MountingHole_2.2mm_M2, F.Cu at (100.0, 57.5)
- added H2: MountingHole, MountingHole:MountingHole_2.2mm_M2, F.Cu at (175.5, 57.0)
- added H3: MountingHole, MountingHole:MountingHole_2.2mm_M2, F.Cu at (176.0, 120.5)
- added H4: MountingHole, MountingHole:MountingHole_2.2mm_M2, F.Cu at (100.5, 121.5)
- added J1: +5V, my_footprints:Terminal_Block_5mm, F.Cu at (108.5, 63.5)
- added J2: EXT_CLK, Connector_PinHeader_2.54mm:PinHeader_1x02_P2.54mm_Vertical, F.Cu at (105.0, 105.8)
- added R1: 100R, Resistor_SMD:R_1206_3216Metric_Pad1.30x1.75mm_HandSolder, F.Cu at (133.6, 76.1)
- added R10: 100R, Resistor_SMD:R_1206_3216Metric_Pad1.30x1.75mm_HandSolder, F.Cu at (169.7, 109.0)
- added R11: 100R, Resistor_SMD:R_1206_3216Metric_Pad1.30x1.75mm_HandSolder, F.Cu at (169.9, 113.5)
- added R12: 100R, Resistor_SMD:R_1206_3216Metric_Pad1.30x1.75mm_HandSolder, F.Cu at (169.9, 117.3)
- added R13: 100R, Resistor_SMD:R_1206_3216Metric_Pad1.30x1.75mm_HandSolder, F.Cu at (164.6, 66.6)
- added R14: 100R, Resistor_SMD:R_1206_3216Metric_Pad1.30x1.75mm_HandSolder, F.Cu at (156.6, 66.6)
- added R15: 1K, Resistor_SMD:R_1206_3216Metric_Pad1.30x1.75mm_HandSolder, F.Cu at (128.1, 113.5)
- added R16: 10K, Resistor_SMD:R_1206_3216Metric_Pad1.30x1.75mm_HandSolder, F.Cu at (128.0, 109.5)
- added R17: 1K, Resistor_SMD:R_1206_3216Metric_Pad1.30x1.75mm_HandSolder, F.Cu at (112.5, 108.6)
- added R18: 10K, Resistor_SMD:R_1206_3216Metric_Pad1.30x1.75mm_HandSolder, F.Cu at (112.5, 102.0)
- added R2: 100R, Resistor_SMD:R_1206_3216Metric_Pad1.30x1.75mm_HandSolder, F.Cu at (133.6, 79.6)
- added R3: 100R, Resistor_SMD:R_1206_3216Metric_Pad1.30x1.75mm_HandSolder, F.Cu at (133.6, 83.1)
- added R4: 100R, Resistor_SMD:R_1206_3216Metric_Pad1.30x1.75mm_HandSolder, F.Cu at (133.6, 86.6)
- added R5: 100R, Resistor_SMD:R_1206_3216Metric_Pad1.30x1.75mm_HandSolder, F.Cu at (133.6, 89.9)
- added R6: 100R, Resistor_SMD:R_1206_3216Metric_Pad1.30x1.75mm_HandSolder, F.Cu at (142.1, 66.6)
- added R7: 100R, Resistor_SMD:R_1206_3216Metric_Pad1.30x1.75mm_HandSolder, F.Cu at (133.7, 72.6)
- added R8: 100R, Resistor_SMD:R_1206_3216Metric_Pad1.30x1.75mm_HandSolder, F.Cu at (169.4, 100.5)
- added R9: 100R, Resistor_SMD:R_1206_3216Metric_Pad1.30x1.75mm_HandSolder, F.Cu at (169.4, 104.4)
- added SW1: EN, my_footprints:slide_switch_2.54mm, F.Cu at (118.5, 105.0)
- added SW2: RST, my_footprints:tact_switch_5mm, F.Cu at (129.0, 102.0)
- added U1: 74LS192, my_footprints:74LS192, F.Cu at (108.3, 83.7)
- added U2: 74LS192, my_footprints:74LS192, F.Cu at (142.8, 106.7)
- added U3: 74LS48, my_footprints:74LS48, F.Cu at (121.3, 83.7)
- added U4: 74LS48, my_footprints:74LS48, F.Cu at (157.5, 107.0)
- added U5: SM420561N, Display_7Segment:7SegmentLED_LTS6760_LTS6780, F.Cu at (141.3, 88.5)
- added U6: SM420561N, Display_7Segment:7SegmentLED_LTS6760_LTS6780, F.Cu at (158.4, 88.3)
Routing:
- net GND: track 0.00 -> 211.8 mm
- net /+5V: track 0.00 -> 161.5 mm, vias 0 -> 4
- net /B0: track 0.00 -> 64.5 mm
- net /Load: track 0.00 -> 61.1 mm, vias 0 -> 1
- net Net-(U6-E): track 0.00 -> 42.3 mm, vias 0 -> 1
- net Net-(U4-f): track 0.00 -> 41.1 mm
- net Net-(U1-QC): track 0.00 -> 40.0 mm
- net Net-(U2-QC): track 0.00 -> 39.5 mm
- net Net-(U4-g): track 0.00 -> 39.2 mm
- net Net-(U6-B): track 0.00 -> 38.1 mm, vias 0 -> 1
- net Net-(U6-D): track 0.00 -> 31.6 mm, vias 0 -> 1
- net /CLK: track 0.00 -> 31.0 mm, vias 0 -> 1
- net Net-(U6-A): track 0.00 -> 30.8 mm, vias 0 -> 1
- net Net-(U2-QD): track 0.00 -> 30.7 mm, vias 0 -> 1
- net Net-(U1-QA): track 0.00 -> 29.5 mm
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Other:
- board outline added: 84.5 x 72.5 mm
- board text added: "24 SECOND COUNTER"
- board text added: "Design Enginneer Jaena,Elaiza Date: 13 Apr 2026"
